File: Version 2/Modular PCB Sets/Southpaw_Split_PCB/Administrative_Button_PCB/Administrative_Button_PCB.kicad_sch (KiCad schematic)
At the start: 17 parts, among them J1 Conn_01x07_Socket

Commit message: created footprints for all lockout and oled display
Parts:
- Tournament_Lockout1: footprint (none) -> Wilson's_Footprint_Library:MTS-101 Toggle Switch
- renumbered D10 to D1, D14 to D2, D15 to D3, D16 to D4, D17 to D5, L3 to L1, R4 to R1, R15 to R2, R16 to R3, R17 to R4, R18 to R5, R3 to R6
Changed lines of the file:
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@@
 		(dnp no)
 		(fields_autoplaced yes)
-		(property "Reference" "R3"
+		(property "Reference" "R6"
 			(at 149.86 113.03 0)
 			(effects
@@
 		)
 		(instances
+			(project "Southpaw_Split_PCB"
+				(path "/12c03e98-16e3-4861-a1ce-d2b4d8ad36ee/e03b2be5-b154-4df2-afd7-f34ad8480ee8"
+					(reference "R6")
+					(unit 1)
+				)
+			)
 			(project "Administrative_Button_PCB"
 				(path "/27e8b247-a568-4b96-98c7-e76fba4b3a84"
@@
 		(dnp no)
 		(fields_autoplaced yes)
-		(property "Reference" "D17"
+		(property "Reference" "D5"
 			(at 129.54 117.1575 0)
 			(effects
@@
 		)
 		(instances
+			(project "Southpaw_Split_PCB"
+				(path "/12c03e98-16e3-4861-a1ce-d2b4d8ad36ee/e03b2be5-b154-4df2-afd7-f34ad8480ee8"
+					(reference "D5")
+					(unit 1)
+				)
+			)
 			(project "Administrative_Button_PCB"
 				(path "/27e8b247-a568-4b96-98c7-e76fba4b3a84"
@@
 		(dnp no)
 		(fields_autoplaced yes)
-		(property "Reference" "R18"
+		(property "Reference" "R5"
 			(at 129.54 107.95 90)
 			(effects
@@
 		)
 		(instances
+			(project "Southpaw_Split_PCB"
+				(path "/12c03e98-16e3-4861-a1ce-d2b4d8ad36ee/e03b2be5-b154-4df2-afd7-f34ad8480ee8"
+					(reference "R5")
+					(unit 1)
+				)
+			)
 			(project "Administrative_Button_PCB"
 				(path "/27e8b247-a568-4b96-98c7-e76fba4b3a84"
@@
 		(on_board yes)
 		(dnp no)
-		(property "Reference" "D14"
+		(property "Reference" "D2"
 			(at 111.76 90.4875 0)
 			(effects
@@
 		)
 		(instances
+			(project "Southpaw_Split_PCB"
+				(path "/12c03e98-16e3-4861-a1ce-d2b4d8ad36ee/e03b2be5-b154-4df2-afd7-f34ad8480ee8"
+					(reference "D2")
+					(unit 1)
+				)
+			)
 			(project "Administrative_Button_PCB"
 				(path "/27e8b247-a568-4b96-98c7-e76fba4b3a84"
@@
 		)
 		(instances
+			(project "Southpaw_Split_PCB"
+				(path "/12c03e98-16e3-4861-a1ce-d2b4d8ad36ee/e03b2be5-b154-4df2-afd7-f34ad8480ee8"
+					(reference "GUIDE1")
+					(unit 1)
+				)
+			)
 			(project "Administrative_Button_PCB"
 				(path "/27e8b247-a568-4b96-98c7-e76fba4b3a84"
@@
 		(dnp no)
 		(fields_autoplaced yes)
-		(property "Reference" "D15"
+		(property "Reference" "D3"
 			(at 116.84 99.3775 0)
 			(effects
@@
 		)
 		(instances
+			(project "Southpaw_Split_PCB"
+				(path "/12c03e98-16e3-4861-a1ce-d2b4d8ad36ee/e03b2be5-b154-4df2-afd7-f34ad8480ee8"
+					(reference "D3")
+					(unit 1)
+				)
+			)
 			(project "Administrative_Button_PCB"
 				(path "/27e8b247-a568-4b96-98c7-e76fba4b3a84"
@@
 		(dnp no)
 		(fields_autoplaced yes)
-		(property "Reference" "R15"
+		(property "Reference" "R2"
 			(at 111.76 81.28 90)
 			(effects
@@
 		)
 		(instances
+			(project "Southpaw_Split_PCB"
+				(path "/12c03e98-16e3-4861-a1ce-d2b4d8ad36ee/e03b2be5-b154-4df2-afd7-f34ad8480ee8"
+					(reference "R2")
+					(unit 1)
+				)
+			)
 			(project "Administrative_Button_PCB"
 				(path "/27e8b247-a568-4b96-98c7-e76fba4b3a84"
@@
 		(dnp no)
 		(fields_autoplaced yes)
-		(property "Reference" "R17"
+		(property "Reference" "R4"
 			(at 121.92 99.06 90)
 			(effects
@@
 		)
 		(instances
+			(project "Southpaw_Split_PCB"
+				(path "/12c03e98-16e3-4861-a1ce-d2b4d8ad36ee/e03b2be5-b154-4df2-afd7-f34ad8480ee8"
+					(reference "R4")
+					(unit 1)
+				)
+			)
 			(project "Administrative_Button_PCB"
 				(path "/27e8b247-a568-4b96-98c7-e76fba4b3a84"
@@
 		(dnp no)
 		(fields_autoplaced yes)
-		(property "Reference" "L3"
+		(property "Reference" "L1"
 			(at 149.86 104.14 0)
 			(effects
@@
 		)
 		(instances
+			(project "Southpaw_Split_PCB"
+				(path "/12c03e98-16e3-4861-a1ce-d2b4d8ad36ee/e03b2be5-b154-4df2-afd7-f34ad8480ee8"
+					(reference "L1")
+					(unit 1)
+				)
+			)
 			(project "Administrative_Button_PCB"
 				(path "/27e8b247-a568-4b96-98c7-e76fba4b3a84"
@@
 		(dnp no)
 		(fields_autoplaced yes)
-		(property "Reference" "R16"
+		(property "Reference" "R3"
 			(at 116.84 90.17 90)
 			(effects
@@
 		)
 		(instances
+			(project "Southpaw_Split_PCB"
+				(path "/12c03e98-16e3-4861-a1ce-d2b4d8ad36ee/e03b2be5-b154-4df2-afd7-f34ad8480ee8"
+					(reference "R3")
+					(unit 1)
+				)
+			)
 			(project "Administrative_Button_PCB"
 				(path "/27e8b247-a568-4b96-98c7-e76fba4b3a84"
@@
 		(dnp no)
 		(fields_autoplaced yes)
-		(property "Reference" "D16"
+		(property "Reference" "D4"
 			(at 121.92 108.2675 0)
 			(effects
@@
 		)
 		(instances
+			(project "Southpaw_Split_PCB"
+				(path "/12c03e98-16e3-4861-a1ce-d2b4d8ad36ee/e03b2be5-b154-4df2-afd7-f34ad8480ee8"
+					(reference "D4")
+					(unit 1)
+				)
+			)
 			(project "Administrative_Button_PCB"
 				(path "/27e8b247-a568-4b96-98c7-e76fba4b3a84"
@@
 		)
 		(instances
+			(project "Southpaw_Split_PCB"
+				(path "/12c03e98-16e3-4861-a1ce-d2b4d8ad36ee/e03b2be5-b154-4df2-afd7-f34ad8480ee8"
+					(reference "BACK1")
+					(unit 1)
+				)
+			)
 			(project "Administrative_Button_PCB"
 				(path "/27e8b247-a568-4b96-98c7-e76fba4b3a84"
@@
 		(dnp no)
 		(fields_autoplaced yes)
-		(property "Reference" "D10"
+		(property "Reference" "D1"
 			(at 106.68 81.5975 0)
 			(effects
@@
 		)
 		(instances
+			(project "Southpaw_Split_PCB"
+				(path "/12c03e98-16e3-4861-a1ce-d2b4d8ad36ee/e03b2be5-b154-4df2-afd7-f34ad8480ee8"
+					(reference "D1")
+					(unit 1)
+				)
+			)
 			(project "Administrative_Button_PCB"
 				(path "/27e8b247-a568-4b96-98c7-e76fba4b3a84"
@@
 			)
 		)
-		(property "Footprint" ""
+		(property "Footprint" "Wilson's_Footprint_Library:MTS-101 Toggle Switch"
 			(at 167.64 120.65 0)
 			(effects
@@
 		)
 		(instances
+			(project "Southpaw_Split_PCB"
+				(path "/12c03e98-16e3-4861-a1ce-d2b4d8ad36ee/e03b2be5-b154-4df2-afd7-f34ad8480ee8"
+					(reference "Tournament_Lockout1")
+					(unit 1)
+				)
+			)
 			(project "Administrative_Button_PCB"
 				(path "/27e8b247-a568-4b96-98c7-e76fba4b3a84"
@@
 		)
 		(instances
+			(project "Southpaw_Split_PCB"
+				(path "/12c03e98-16e3-4861-a1ce-d2b4d8ad36ee/e03b2be5-b154-4df2-afd7-f34ad8480ee8"
+					(reference "START1")
+					(unit 1)
+				)
+			)
 			(project "Administrative_Button_PCB"
 				(path "/27e8b247-a568-4b96-98c7-e76fba4b3a84"
@@
 		(dnp no)
 		(fields_autoplaced yes)
-		(property "Reference" "R4"
+		(property "Reference" "R1"
 			(at 106.68 72.39 90)
 			(effects
@@
 		)
 		(instances
-			(project "Administrative_Button_PCB"
-				(path "/27e8b247-a568-4b96-98c7-e76fba4b3a84"
+			(project "Southpaw_Split_PCB"
+				(path "/12c03e98-16e3-4861-a1ce-d2b4d8ad36ee/e03b2be5-b154-4df2-afd7-f34ad8480ee8"
+					(reference "R1")
+					(unit 1)
+				)
+			)
+			(project "Administrative_Button_PCB"
+				(path "/27e8b247-a568-4b96-98c7-e76fba4b3a84"

Commit message: general part layout
Parts:
- renumbered L1 to L3SW1, R6 to R3SW1
Other:
- moved on the sheet: BACK1, D1, GUIDE1, J1, L3SW1, R1, R3SW1, START1, Tournament_Lockout1
