File: Version 2/Modular PCB Sets/Southpaw_Split_PCB/Southpaw_Split_PCB.kicad_pcb (KiCad board)
At the start: 2 copper layers, 254 x 112 mm, 56 parts, among them J1 Conn_01x06_Socket, J1 Conn_01x07_Socket, J2 Conn_01x07_Socket, U1 Pico, X1 SW_SPST, Y1 SW_SPST

Commit message: created footprints for all lockout and oled display
Parts:
- removed the J1 at (126.0, 51.0)
- removed the J1 at (156.0, 77.0)
- removed J2: Conn_01x07_Socket, Connector_JST:JST_PH_B7B-PH-K_1x07_P2.00mm_Vertical
- removed U1: Pico, Module:RaspberryPi_Pico_Common_THT
- added A2: RaspberryPi_Pico, Module:RaspberryPi_Pico_Common_Unspecified, F.Cu at (91.6, 167.1)
- added J1: Conn_01x06_Socket, Connector_JST:JST_PH_B6B-PH-K_1x06_P2.00mm_Vertical, B.Cu at (151.0, 136.0)
- added J1: Conn_01x07_Socket, Connector_JST:JST_PH_B7B-PH-K_1x07_P2.00mm_Vertical, B.Cu at (34.0, 41.0)
- added J1: Conn_01x07_Socket, Connector_JST:JST_PH_B7B-PH-K_1x07_P2.00mm_Vertical, B.Cu at (119.0, 29.0)
- added J4: Conn_01x07_Socket, Connector_JST:JST_PH_B7B-PH-K_1x07_P2.00mm_Vertical, B.Cu at (153.0, 81.0)
- added J5: Conn_01x07_Socket, Connector_JST:JST_PH_B7B-PH-K_1x07_P2.00mm_Vertical, B.Cu at (28.0, 82.0)
- added SW1: RotaryEncoder_Switch, Rotary_Encoder:RotaryEncoder_Alps_EC11E-Switch_Vertical_H20mm, F.Cu at (32.5, 50.5)
- added Tournament_Lockout1: SW_SPST, Wilson's_Footprint_Library:MTS-101 Toggle Switch, F.Cu at (124.5, 39.0)
- added U2: ~, Wilson's_Footprint_Library:Hosyond SH1106 OLED Display, F.Cu at (50.4, 59.8)
- moved D1 16.3 mm to (68.0, 88.0)
- moved D2 16.3 mm to (35.5, 96.0)
- moved D3 16.3 mm to (97.5, 85.0)
- moved D4 16.3 mm to (131.5, 93.0)
- moved D5 16.3 mm to (38.5, 132.0)
- moved D6 16.3 mm to (68.5, 124.0)
- moved D7 16.3 mm to (96.5, 122.0)
- moved D8 16.3 mm to (130.5, 127.0)
- moved LB1 16.3 mm to (39.5, 103.9)
- moved R1 16.3 mm to (137.0, 128.0)
- moved R10 16.3 mm to (73.9, 89.0)
- moved R11 16.3 mm to (42.0, 97.0)
- moved R5 16.3 mm to (103.0, 123.0)
- moved R6 16.3 mm to (74.8, 125.0)
- moved R7 16.3 mm to (44.9, 132.0)
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Routing:
- net /Gnd: track 158.5 -> 573.5 mm
- net GND: track 0.00 -> 238.2 mm
- net 3v3: track 0.00 -> 236.1 mm
- net /Rotary_Encoder_DT: track 0.00 -> 180.0 mm, vias 0 -> 2
- net /Rotary_Encoder_CLK: track 0.00 -> 170.2 mm, vias 0 -> 1
- net /SDA: track 0.00 -> 154.5 mm
- net /SCK: track 0.00 -> 151.7 mm
- net /Encoder_Press: track 0.00 -> 149.7 mm
- net LB: track 0.00 -> 149.7 mm, vias 0 -> 1
- net Net-(BACK1-B): track 123.5 -> 0.00 mm
- net /Right: track 97.2 -> 208.8 mm, vias 0 -> 2
- net RB: track 0.00 -> 111.4 mm
- net /3V3: track 174.7 -> 280.2 mm
- net X: track 0.00 -> 101.7 mm
- net Y: track 0.00 -> 101.4 mm
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Other:
- board size 254 x 112 mm -> 260 x 168 mm

Commit message: general part layout
Parts:
- removed the D1 at (68.0, 88.0)
- removed D10, D14, D15, D16, D17: LED, LED_THT:LED_D5.0mm
- removed the D2 at (35.5, 96.0)
- removed the D3 at (97.5, 85.0)
- removed the D4 at (131.5, 93.0)
- removed the D5 at (38.5, 132.0)
- removed the J1 at (151.0, 136.0)
- removed the J1 at (34.0, 41.0)
- removed the J1 at (119.0, 29.0)
- removed the J1 at (174.0, 77.0)
- removed J4, J5: Conn_01x07_Socket, Connector_JST:JST_PH_B7B-PH-K_1x07_P2.00mm_Vertical
- removed L3: SW_SPST, Button_Switch_Keyboard:SW_Cherry_MX_1.00u_PCB
- removed the R1 at (137.0, 128.0)
- removed R10, R11, R15, R16, R17, R18, R9: R, Resistor_THT:R_Axial_DIN0207_L6.3mm_D2.5mm_P10.16mm_Horizontal
- removed the R2 at (189.8, 126.0)
- removed the R3 at (262.5, 29.9)
- removed the R4 at (160.9, 34.9)
- removed the R5 at (103.0, 123.0)
- removed SW1: RotaryEncoder_Switch, Rotary_Encoder:RotaryEncoder_Alps_EC11E-Switch_Vertical_H20mm
- removed U2: ~, Wilson's_Footprint_Library:Hosyond SH1106 OLED Display
- added D1: LED, LED_THT:LED_D5.0mm, F.Cu at (69.5, 33.0)
- added D1: LED, LED_THT:LED_D5.0mm, F.Cu at (133.0, 121.0)
- added D2: LED, LED_THT:LED_D5.0mm, F.Cu at (97.5, 33.0)
- added D2: LED, LED_THT:LED_D5.0mm, F.Cu at (99.0, 116.0)
- added D3: LED, LED_THT:LED_D5.0mm, F.Cu at (71.5, 118.0)
- added D3: LED, LED_THT:LED_D5.0mm, F.Cu at (125.5, 33.0)
- added D4: LED, LED_THT:LED_D5.0mm, F.Cu at (41.0, 126.0)
- added D4: LED, LED_THT:LED_D5.0mm, F.Cu at (153.5, 33.0)
- added D5: LED, LED_THT:LED_D5.0mm, F.Cu at (181.5, 33.0)
- added D5: LED, LED_THT:LED_D5.0mm, F.Cu at (135.0, 87.0)
- added J1: Conn_01x06_Socket, Connector_JST:JST_PH_B6B-PH-K_1x06_P2.00mm_Vertical, B.Cu at (156.0, 139.0)
- added J1: Conn_01x06_Socket, Connector_JST:JST_PH_B6B-PH-K_1x06_P2.00mm_Vertical, B.Cu at (172.0, 125.0)
- added J1: Conn_01x07_Socket, Connector_JST:JST_PH_B7B-PH-K_1x07_P2.00mm_Vertical, B.Cu at (42.0, 45.0)
- added J2: Conn_01x07_Socket, Connector_JST:JST_PH_B7B-PH-K_1x07_P2.00mm_Vertical, B.Cu at (156.0, 75.0)
- added J3: Conn_01x07_Socket, Connector_JST:JST_PH_B7B-PH-K_1x07_P2.00mm_Vertical, B.Cu at (221.0, 56.0)
- added J3: Conn_01x07_Socket, Connector_JST:JST_PH_B7B-PH-K_1x07_P2.00mm_Vertical, B.Cu at (43.0, 75.0)
- added L3SW1: SW_SPST, Button_Switch_Keyboard:SW_Cherry_MX_1.00u_PCB, F.Cu at (171.5, 32.9)
- added OLED1: ~, Wilson's_Footprint_Library:Hosyond SH1106 OLED Display, F.Cu at (226.3, 58.8)
- added R1: R, Resistor_THT:R_Axial_DIN0207_L6.3mm_D2.5mm_P10.16mm_Horizontal, F.Cu at (71.0, 38.9)
- added R1: R, Resistor_THT:R_Axial_DIN0207_L6.3mm_D2.5mm_P10.16mm_Horizontal, F.Cu at (138.9, 122.0)
- added R2: R, Resistor_THT:R_Axial_DIN0207_L6.3mm_D2.5mm_P10.16mm_Horizontal, F.Cu at (105.4, 117.0)
- added R2: R, Resistor_THT:R_Axial_DIN0207_L6.3mm_D2.5mm_P10.16mm_Horizontal, F.Cu at (187.8, 145.0)
- added R2: R, Resistor_THT:R_Axial_DIN0207_L6.3mm_D2.5mm_P10.16mm_Horizontal, F.Cu at (99.0, 38.9)
- added R3: R, Resistor_THT:R_Axial_DIN0207_L6.3mm_D2.5mm_P10.16mm_Horizontal, F.Cu at (77.8, 119.0)
- added R3: R, Resistor_THT:R_Axial_DIN0207_L6.3mm_D2.5mm_P10.16mm_Horizontal, F.Cu at (127.0, 38.9)
- added R3SW1: SW_SPST, Button_Switch_Keyboard:SW_Cherry_MX_1.00u_PCB, F.Cu at (143.5, 32.9)
- added R4: R, Resistor_THT:R_Axial_DIN0207_L6.3mm_D2.5mm_P10.16mm_Horizontal, F.Cu at (47.4, 127.0)
- added R4: R, Resistor_THT:R_Axial_DIN0207_L6.3mm_D2.5mm_P10.16mm_Horizontal, F.Cu at (155.0, 38.9)
- added R5: R, Resistor_THT:R_Axial_DIN0207_L6.3mm_D2.5mm_P10.16mm_Horizontal, F.Cu at (141.4, 87.0)
- added R5: R, Resistor_THT:R_Axial_DIN0207_L6.3mm_D2.5mm_P10.16mm_Horizontal, F.Cu at (182.0, 38.9)
- added RotarySW1: RotaryEncoder_Switch, Rotary_Encoder:RotaryEncoder_Alps_EC11E-Switch_Vertical_H20mm, F.Cu at (203.5, 40.0)
- moved D8 99.2 mm to (38.5, 90.0)
- moved Tournament_Lockout1 95.9 mm to (28.6, 37.9)
- moved R8 93.1 mm to (44.8, 91.0)
- moved GUIDE1 92.1 mm to (115.5, 32.9)
- moved BACK1 91.9 mm to (87.5, 32.9)
- moved START1 91.1 mm to (59.5, 32.9)
- moved R7 58.5 mm to (76.9, 83.0)
- moved R6 55.3 mm to (106.9, 80.0)
- moved D6 55.2 mm to (100.5, 79.0)
- moved D7 47.8 mm to (70.5, 82.0)
- moved R14 22.6 mm to (198.9, 106.0), turned to 0 degrees
- moved D12 19.1 mm to (222.2, 89.5)
- moved D13 19.1 mm to (258.1, 97.5)
- moved D9 19.1 mm to (194.1, 108.5)
- moved DOWN1 19.1 mm to (224.5, 95.9)
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Connections:
- D6 pad 1: RT -> Y
- D7 pad 1: B -> RB
- D8 pad 1: A -> LB
- R7 pad 1: Net-(D5-A) -> Net-(D7-A)
- R8 pad 1: Net-(D4-A) -> Net-(D8-A)
Routing:
- net /Gnd: track 573.5 -> 0.00 mm
- net /3V3: track 280.2 -> 0.00 mm
- net GND: track 238.2 -> 0.00 mm
- net 3v3: track 236.1 -> 0.00 mm
- net /Right: track 208.8 -> 0.00 mm, vias 2 -> 0
- net /Rotary_Encoder_DT: track 180.0 -> 0.00 mm, vias 2 -> 0
- net /Rotary_Encoder_CLK: track 170.2 -> 0.00 mm, vias 1 -> 0
- net /Up: track 167.3 -> 0.00 mm
- net /SDA: track 154.5 -> 0.00 mm
- net /SCK: track 151.7 -> 0.00 mm
- net /Encoder_Press: track 149.7 -> 0.00 mm
- net LB: track 149.7 -> 0.00 mm, vias 1 -> 0
- net /Down: track 149.7 -> 0.00 mm, vias 1 -> 0
- net /R3: track 147.1 -> 0.00 mm, vias 2 -> 0
- net /L3: track 142.6 -> 0.00 mm, vias 2 -> 0
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Other:
- board size 260 x 168 mm -> 255 x 163 mm

Commit message: Finalized design and uploaded gerbers to JLCpcb, waiting for boards to come in
Parts:
- removed the D1 at (69.5, 33.0)
- removed the D1 at (133.0, 121.0)
- removed D11, D12, D13: LED, LED_THT:LED_D5.0mm
- removed the D2 at (97.5, 33.0)
- removed the D2 at (99.0, 116.0)
- removed the D3 at (71.5, 118.0)
- removed the D3 at (125.5, 33.0)
- removed the D4 at (41.0, 126.0)
- removed the D4 at (153.5, 33.0)
- removed the D5 at (181.5, 33.0)
- removed the D5 at (135.0, 87.0)
- removed the D6 at (100.5, 79.0)
- removed the D7 at (70.5, 82.0)
- removed the D8 at (38.5, 90.0)
- removed the J1 at (156.0, 139.0)
- removed the J1 at (172.0, 125.0)
- removed the J1 at (42.0, 45.0)
- removed the J3 at (221.0, 56.0)
- removed the J3 at (43.0, 75.0)
- removed the R1 at (71.0, 38.9)
- removed the R1 at (138.9, 122.0)
- removed R12, R13, R14: R, Resistor_THT:R_Axial_DIN0207_L6.3mm_D2.5mm_P10.16mm_Horizontal
- removed the R2 at (105.4, 117.0)
- removed the R2 at (187.8, 145.0)
- removed the R2 at (99.0, 38.9)
- removed the R3 at (77.8, 119.0)
- removed the R3 at (127.0, 38.9)
- removed the R4 at (47.4, 127.0)
- removed the R4 at (155.0, 38.9)
- removed the R5 at (141.4, 87.0)
- removed the R5 at (182.0, 38.9)
- removed the R6 at (106.9, 80.0)
- removed the R7 at (76.9, 83.0)
- removed the R8 at (44.8, 91.0)
- added D1: LED, LED_THT:LED_D5.0mm, F.Cu at (146.7, 21.0)
- added D1: LED, LED_THT:LED_D5.0mm, F.Cu at (144.9, 122.2)
- added D2: LED, LED_THT:LED_D5.0mm, F.Cu at (111.3, 112.2)
- added D2: LED, LED_THT:LED_D5.0mm, F.Cu at (116.7, 21.0)
- added D3: LED, LED_THT:LED_D5.0mm, F.Cu at (76.9, 118.2)
- added D3: LED, LED_THT:LED_D5.0mm, F.Cu at (86.7, 21.0)
- added D4: LED, LED_THT:LED_D5.0mm, F.Cu at (42.6, 125.2)
- added D4: LED, LED_THT:LED_D5.0mm, F.Cu at (26.7, 21.0)
- added D5: LED, LED_THT:LED_D5.0mm, F.Cu at (144.9, 87.2)
- added D5: LED, LED_THT:LED_D5.0mm, F.Cu at (56.7, 21.0)
- added D6: LED, LED_THT:LED_D5.0mm, F.Cu at (194.7, 141.6)
- added D6: LED, LED_THT:LED_D5.0mm, F.Cu at (111.3, 77.2)
- added D7: LED, LED_THT:LED_D5.0mm, F.Cu at (227.7, 75.0)
- added D7: LED, LED_THT:LED_D5.0mm, F.Cu at (76.9, 83.2)
- added D8: LED, LED_THT:LED_D5.0mm, F.Cu at (257.7, 74.0)
- added D8: LED, LED_THT:LED_D5.0mm, F.Cu at (42.6, 90.2)
- added J1: Conn_01x06_Socket, Connector_JST:JST_PH_B6B-PH-K_1x06_P2.00mm_Vertical, B.Cu at (162.2, 168.2)
- added J1: Conn_01x07_Socket, Connector_JST:JST_PH_B7B-PH-K_1x07_P2.00mm_Vertical, B.Cu at (184.0, 39.5)
- added J3: Conn_01x07_Socket, Connector_JST:JST_PH_B7B-PH-K_1x07_P2.00mm_Vertical, B.Cu at (230.4, 45.4)
- added J3: Conn_01x07_Socket, Connector_JST:JST_PH_B7B-PH-K_1x07_P2.00mm_Vertical, B.Cu at (40.5, 78.2)
- added J6: Conn_01x06_Socket, Connector_JST:JST_PH_B6B-PH-K_1x06_P2.00mm_Vertical, B.Cu at (181.3, 132.1)
- added R1: R, Resistor_THT:R_Axial_DIN0207_L6.3mm_D2.5mm_P10.16mm_Horizontal, F.Cu at (151.4, 122.2)
- added R1: R, Resistor_THT:R_Axial_DIN0207_L6.3mm_D2.5mm_P10.16mm_Horizontal, F.Cu at (153.3, 21.0)
- added R2: R, Resistor_THT:R_Axial_DIN0207_L6.3mm_D2.5mm_P10.16mm_Horizontal, F.Cu at (123.3, 21.0)
- added R2: R, Resistor_THT:R_Axial_DIN0207_L6.3mm_D2.5mm_P10.16mm_Horizontal, F.Cu at (117.9, 112.2)
- added R3: R, Resistor_THT:R_Axial_DIN0207_L6.3mm_D2.5mm_P10.16mm_Horizontal, F.Cu at (93.3, 21.0)
- added R3: R, Resistor_THT:R_Axial_DIN0207_L6.3mm_D2.5mm_P10.16mm_Horizontal, F.Cu at (83.4, 118.2)
- added R4: R, Resistor_THT:R_Axial_DIN0207_L6.3mm_D2.5mm_P10.16mm_Horizontal, F.Cu at (49.1, 125.2)
- added R4: R, Resistor_THT:R_Axial_DIN0207_L6.3mm_D2.5mm_P10.16mm_Horizontal, F.Cu at (33.3, 21.0)
- added R5: R, Resistor_THT:R_Axial_DIN0207_L6.3mm_D2.5mm_P10.16mm_Horizontal, F.Cu at (151.4, 87.2)
- added R5: R, Resistor_THT:R_Axial_DIN0207_L6.3mm_D2.5mm_P10.16mm_Horizontal, F.Cu at (63.3, 21.0)
- added R6: R, Resistor_THT:R_Axial_DIN0207_L6.3mm_D2.5mm_P10.16mm_Horizontal, F.Cu at (201.3, 141.6)
- added R6: R, Resistor_THT:R_Axial_DIN0207_L6.3mm_D2.5mm_P10.16mm_Horizontal, F.Cu at (117.9, 77.2)
- added R7: R, Resistor_THT:R_Axial_DIN0207_L6.3mm_D2.5mm_P10.16mm_Horizontal, F.Cu at (83.4, 83.2)
- added R7: R, Resistor_THT:R_Axial_DIN0207_L6.3mm_D2.5mm_P10.16mm_Horizontal, F.Cu at (234.3, 75.0)
- added R8: R, Resistor_THT:R_Axial_DIN0207_L6.3mm_D2.5mm_P10.16mm_Horizontal, F.Cu at (49.1, 90.2)
- added R8: R, Resistor_THT:R_Axial_DIN0207_L6.3mm_D2.5mm_P10.16mm_Horizontal, F.Cu at (264.3, 74.0)
- added R9: R, Resistor_THT:R_Axial_DIN0207_L6.3mm_D2.5mm_P10.16mm_Horizontal, F.Cu at (209.3, 91.6)
- moved Tournament_Lockout1 156.9 mm to (184.5, 20.0), turned to 180 degrees
- moved L3SW1 141.0 mm to (30.5, 26.9)
- moved START1 91.3 mm to (150.5, 26.9)
- moved R3SW1 83.1 mm to (60.5, 26.9)
- moved BACK1 33.5 mm to (120.5, 26.9)
- moved GUIDE1 25.6 mm to (90.5, 26.9)
- moved RIGHT1 24.0 mm to (261.5, 79.9)
- moved LEFT1 20.0 mm to (206.5, 97.5)
- moved D9 19.0 mm to (202.7, 91.6), turned to 0 degrees
- moved RotarySW1 18.1 mm to (221.6, 39.1), turned to 90 degrees
- moved OLED1 16.7 mm to (239.7, 48.7)
- moved DOWN1 16.6 mm to (231.5, 80.9)
- moved UP1 14.2 mm to (198.5, 147.5)
- moved B1 13.1 mm to (115.2, 118.1)
- moved Y1 11.4 mm to (115.2, 83.1)
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Connections:
- A2 pad 13: /Gnd -> GND
- A2 pad 18: /Gnd -> GND
- A2 pad 23: /Gnd -> GND
- A2 pad 28: /Gnd -> GND
- A2 pad 3: /Gnd -> GND
- A2 pad 36: /3V3 -> 3v3
- A2 pad 38: /Gnd -> GND
- A2 pad 8: /Gnd -> GND
- J2 pad 1: /Gnd -> GND
- J2 pad 2: /3V3 -> 3v3
Routing:
- net GND: track 0.00 -> 469.0 mm
- net 3v3: track 0.00 -> 446.5 mm
- net Net-(BACK1-B): track 0.00 -> 286.1 mm
- net /L3: track 0.00 -> 277.7 mm
- net /R3: track 0.00 -> 268.7 mm
- net /Guide: track 0.00 -> 224.7 mm
- net /Right: track 0.00 -> 214.4 mm
- net /3V3: track 0.00 -> 213.6 mm
- net /SDA: track 0.00 -> 211.0 mm, vias 0 -> 2
- net /Gnd: track 0.00 -> 208.0 mm
- net /SCK: track 0.00 -> 207.4 mm
- net /Options: track 0.00 -> 177.2 mm
- net /3v3: track 0.00 -> 156.3 mm
- net /Start: track 0.00 -> 154.8 mm
- net /Down: track 0.00 -> 149.7 mm
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Other:
- board size 255 x 163 mm -> 280.2 x 171 mm
